Commit message: run ok but not completed: map & navi

File: dev_ws/src/articubot_one/description/lidar.xacro (robot description, xacro)
@@ -14,9 +14,9 @@
         <material name="red"/>
     </visual>
-    <collision>
+    <!-- <collision>
         <geometry>
             <cylinder radius="0.05" length="0.04"/>
         </geometry>
-    </collision>
+    </collision> -->
     <xacro:inertial_cylinder mass="0.1" length="0.04" radius="0.05">
         <!-- <origin xyz="0.21 0 0.25" rpy="0 0 0"/> -->
@@ -39,6 +39,6 @@
                 </scan>
                 <range>
-                    <min>0.1</min>
-                    <max>40.0</max>
+                    <min>0.3</min>
+                    <max>10.0</max>
                 </range>
             </ray>

Commit message: add node camera

File: dev_ws/src/articubot_one/description/lidar.xacro (robot description, xacro)
@@ -5,5 +5,5 @@
         <child link="laser_frame"/>
         <!-- <origin xyz="0.21 0 0.25" rpy="0 0 0"/> -->
-        <origin xyz="0.21 0 0.05" rpy="0 0 3.1415926535"/>
+            <origin xyz="0.21 0 0.16" rpy="0 0 3.1415926535"/>
     </joint>
     <link name="laser_frame">

File: dev_ws/src/articubot_one/description/robot.urdf.xacro (robot description, xacro)
@@ -4,4 +4,4 @@
     <xacro:include filename="gazebo_control.xacro" />
     <xacro:include filename="lidar.xacro" />
-    <!-- <xacro:include filename="camera.xacro" /> -->
+    <xacro:include filename="camera.xacro" />
 </robot>

File: dev_ws/src/articubot_one/description/robot_core.xacro (robot description, xacro)
@@ -32,28 +32,22 @@
         <parent link="base_link"/>
         <child link="chassis"/>
-        <origin xyz="-0.1 0 0"/>
+        <origin xyz="0 0 0"/>
     </joint>
     <link name="chassis">
         <visual>
-            <!-- <origin xyz="0.15 0 0.075"/> -->
-            <origin xyz="0.15 0 0.015"/>
+            <origin xyz="0.13 0 0.07"/>
             <geometry>
-                <!-- <box size="0.3 0.3 0.15"/> -->
-                <box size="0.3 0.3 0.03"/>
+                <box size="0.26 0.20 0.06"/>
             </geometry>
             <material name="white"/>
         </visual>
         <collision>
-            <!-- <origin xyz="0.15 0 0.075"/> -->
-            <origin xyz="0.15 0 0.015"/>
+            <origin xyz="0.13 0 0.07"/>
             <geometry>
-                <!-- <box size="0.3 0.3 0.15"/> -->
-                <box size="0.3 0.3 0.03"/>
+                <box size="0.26 0.20 0.06"/>
             </geometry>
         </collision>
-        <!-- <xacro:inertial_box mass="0.5" x="0.3" y="0.3" z="0.15"> -->
-        <xacro:inertial_box mass="0.5" x="0.3" y="0.3" z="0.03">
-            <!-- <origin xyz="0.15 0 0.075" rpy="0 0 0"/> -->
-            <origin xyz="0.15 0 0.015" rpy="0 0 0"/>
+        <xacro:inertial_box mass="0.5" x="0.26" y="0.20" z="0.06">
+            <origin xyz="0.13 0 0.07" rpy="0 0 0"/>
         </xacro:inertial_box>
     </link>
@@ -65,5 +59,5 @@
         <parent link="base_link"/>
         <child link="left_wheel"/>
-        <origin xyz="0 0.175 0" rpy="-${pi/2} 0 0" />
+        <origin xyz="0 0.13 0" rpy="-${pi/2} 0 0" />
         <axis xyz="0 0 1"/>
     </joint>
@@ -71,5 +65,5 @@
         <visual>
             <geometry>
-                <cylinder radius="0.034" length="0.04"/>
+                <cylinder radius="0.034" length="0.02"/>
             </geometry>
             <material name="blue"/>
@@ -77,8 +71,8 @@
         <collision>
             <geometry>
-                <cylinder radius="0.034" length="0.04"/>
+                <cylinder radius="0.034" length="0.02"/>
             </geometry>
         </collision>
-        <xacro:inertial_cylinder mass="0.1" length="0.04" radius="0.05">
+        <xacro:inertial_cylinder mass="0.1" length="0.02" radius="0.034">
             <origin xyz="0 0 0" rpy="0 0 0"/>
         </xacro:inertial_cylinder>
@@ -91,5 +85,5 @@
         <parent link="base_link"/>
         <child link="right_wheel"/>
-        <origin xyz="0 -0.175 0" rpy="${pi/2} 0 0" />
+        <origin xyz="0 -0.13 0" rpy="${pi/2} 0 0" />
         <axis xyz="0 0 -1"/>
     </joint>
@@ -97,5 +91,5 @@
         <visual>
             <geometry>
-                <cylinder radius="0.034" length="0.04"/>
+                <cylinder radius="0.034" length="0.02"/>
             </geometry>
             <material name="blue"/>
@@ -103,8 +97,8 @@
         <collision>
             <geometry>
-                <cylinder radius="0.034" length="0.04"/>
+                <cylinder radius="0.034" length="0.02"/>
             </geometry>
         </collision>
-        <xacro:inertial_cylinder mass="0.1" length="0.04" radius="0.05">
+        <xacro:inertial_cylinder mass="0.1" length="0.02" radius="0.02">
             <origin xyz="0 0 0" rpy="0 0 0"/>
         </xacro:inertial_cylinder>
@@ -117,5 +111,5 @@
         <parent link="chassis"/>
         <child link="caster_wheel"/>
-        <origin xyz="0.24 0 0"/>
+        <origin xyz="0.21 0 0"/>
     </joint>
     <link name="caster_wheel">
@@ -128,5 +122,5 @@
         <collision>
             <geometry>
-                <sphere radius="0.03"/>
+                <sphere radius="0.05"/>
             </geometry>
         </collision>

Commit message: fix navigation in real robot

File: dev_ws/src/articubot_one/description/lidar.xacro (robot description, xacro)
@@ -4,5 +4,5 @@
         <parent link="chassis"/>
         <child link="laser_frame"/>
-            <origin xyz="0.21 0 0.16" rpy="0 0 0"/>
+            <origin xyz="0.21 0 0.16" rpy="0 0 3.1415926535"/>
     </joint>
     <link name="laser_frame">
@@ -26,5 +26,5 @@
     </collision>
     <xacro:inertial_cylinder mass="0.1" length="0.04" radius="0.05">
-        <origin xyz="0 0 0" rpy="0 0 0"/>
+        <origin xyz="0 0 0" rpy="0 0 3.1415926535"/>
     </xacro:inertial_cylinder>
     </link>
